Commit message: Change mesh paths to gazebo format

File: robot_control_assets/assets/arms/panda/panda.urdf (robot description, URDF)
Before this commit: robot panda, 13 links, 12 joints
Links:
- link panda_hand: geometry collision mesh filename=package://robot_control_assets/assets/arms/panda/meshes/col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; visual mesh filename=package://robot_control_assets/assets/arms/panda/meshes/vis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
- link panda_leftfinger: geometry collision mesh filename=package://robot_control_assets/assets/arms/panda/meshes/col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; visual mesh filename=package://robot_control_assets/assets/arms/panda/meshes/vis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
- link panda_link0: geometry collision mesh filename=package://robot_control_assets/assets/arms/panda/meshes/col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; visual mesh filename=package://robot_control_assets/assets/arms/panda/meshes/vis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
- link panda_link1: geometry collision mesh filename=package://robot_control_assets/assets/arms/panda/meshes/col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; visual mesh filename=package://robot_control_assets/assets/arms/panda/meshes/vis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
- link panda_link2: geometry collision mesh filename=package://robot_control_assets/assets/arms/panda/meshes/col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; visual mesh filename=package://robot_control_assets/assets/arms/panda/meshes/vis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
- link panda_link3: geometry collision mesh filename=package://robot_control_assets/assets/arms/panda/meshes/col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; visual mesh filename=package://robot_control_assets/assets/arms/panda/meshes/vis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
- link panda_link4: geometry collision mesh filename=package://robot_control_assets/assets/arms/panda/meshes/col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; visual mesh filename=package://robot_control_assets/assets/arms/panda/meshes/vis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
- link panda_link5: geometry collision mesh filename=package://robot_control_assets/assets/arms/panda/meshes/col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; visual mesh filename=package://robot_control_assets/assets/arms/panda/meshes/vis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
- link panda_link6: geometry collision mesh filename=package://robot_control_assets/assets/arms/panda/meshes/col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; visual mesh filename=package://robot_control_assets/assets/arms/panda/meshes/vis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
- link panda_link7: geometry collision mesh filename=package://robot_control_assets/assets/arms/panda/meshes/col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; visual mesh filename=package://robot_control_assets/assets/arms/panda/meshes/vis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
- link panda_rightfinger: geometry collision mesh filename=package://robot_control_assets/assets/arms/panda/meshes/col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; visual mesh filename=package://robot_control_assets/assets/arms/panda/meshes/vis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
