Commit message: Run panda urdf through xacro for gazebo compatibility

File: robot_control_assets/assets/arms/panda/panda.urdf.xacro (robot description, xacro)
@@ -1,9 +1,7 @@
 <?xml version="1.0" encoding="utf-8"?>
-<!-- =================================================================================== -->
-<!-- |    This document was autogenerated by xacro from panda_arm_hand.urdf.xacro      | -->
-<!-- |    EDITING THIS FILE BY HAND IS NOT RECOMMENDED                                 | -->
-<!-- =================================================================================== -->
 <robot name="panda" xmlns:xacro="http://www.ros.org/wiki/xacro">
   <xacro:property name="joint_damping" value="1.0"/>
+  <xacro:arg name="mesh_prefix" default="model://" />
+  <xacro:property name="mesh_prefix" value="$(arg mesh_prefix)" />
   <link name="world"/>
   <joint name="panda_joint_world" type="fixed">
@@ -135,14 +133,14 @@
       <origin rpy="0 0 0" xyz="0 0 0"/>
       <geometry>
-        <mesh filename="package://robot_control_assets/assets/arms/panda/meshes/visual/link0.dae"/>
-      </geometry>
-      <material name="">
-        <color rgba="1 1 1 1"/>
-      </material>
-    </visual>
-    <collision>
-      <origin rpy="0 0 0" xyz="0 0 0"/>
-      <geometry>
-        <mesh filename="package://robot_control_assets/assets/arms/panda/meshes/collision/link0.stl"/>
+        <mesh filename="${mesh_prefix}assets/arms/panda/meshes/visual/link0.dae"/>
+      </geometry>
+      <material name="">
+        <color rgba="1 1 1 1"/>
+      </material>
+    </visual>
+    <collision>
+      <origin rpy="0 0 0" xyz="0 0 0"/>
+      <geometry>
+        <mesh filename="${mesh_prefix}assets/arms/panda/meshes/collision/link0.stl"/>
       </geometry>
     </collision>
@@ -157,14 +155,14 @@
       <origin rpy="0 0 0" xyz="0 0 0"/>
       <geometry>
-        <mesh filename="package://robot_control_assets/assets/arms/panda/meshes/visual/link1.dae"/>
-      </geometry>
-      <material name="">
-        <color rgba="1 1 1 1"/>
-      </material>
-    </visual>
-    <collision>
-      <origin rpy="0 0 0" xyz="0 0 0"/>
-      <geometry>
-        <mesh filename="package://robot_control_assets/assets/arms/panda/meshes/collision/link1.stl"/>
+        <mesh filename="${mesh_prefix}assets/arms/panda/meshes/visual/link1.dae"/>
+      </geometry>
+      <material name="">
+        <color rgba="1 1 1 1"/>
+      </material>
+    </visual>
+    <collision>
+      <origin rpy="0 0 0" xyz="0 0 0"/>
+      <geometry>
+        <mesh filename="${mesh_prefix}assets/arms/panda/meshes/collision/link1.stl"/>
       </geometry>
     </collision>
@@ -188,14 +186,14 @@
       <origin rpy="0 0 0" xyz="0 0 0"/>
       <geometry>
-        <mesh filename="package://robot_control_assets/assets/arms/panda/meshes/visual/link2.dae"/>
-      </geometry>
-      <material name="">
-        <color rgba="1 1 1 1"/>
-      </material>
-    </visual>
-    <collision>
-      <origin rpy="0 0 0" xyz="0 0 0"/>
-      <geometry>
-        <mesh filename="package://robot_control_assets/assets/arms/panda/meshes/collision/link2.stl"/>
+        <mesh filename="${mesh_prefix}assets/arms/panda/meshes/visual/link2.dae"/>
+      </geometry>
+      <material name="">
+        <color rgba="1 1 1 1"/>
+      </material>
+    </visual>
+    <collision>
+      <origin rpy="0 0 0" xyz="0 0 0"/>
+      <geometry>
+        <mesh filename="${mesh_prefix}assets/arms/panda/meshes/collision/link2.stl"/>
       </geometry>
     </collision>
@@ -219,14 +217,14 @@
       <origin rpy="0 0 0" xyz="0 0 0"/>
       <geometry>
-        <mesh filename="package://robot_control_assets/assets/arms/panda/meshes/visual/link3.dae"/>
-      </geometry>
-      <material name="">
-        <color rgba="1 1 1 1"/>
-      </material>
-    </visual>
-    <collision>
-      <origin rpy="0 0 0" xyz="0 0 0"/>
-      <geometry>
-        <mesh filename="package://robot_control_assets/assets/arms/panda/meshes/collision/link3.stl"/>
+        <mesh filename="${mesh_prefix}assets/arms/panda/meshes/visual/link3.dae"/>
+      </geometry>
+      <material name="">
+        <color rgba="1 1 1 1"/>
+      </material>
+    </visual>
+    <collision>
+      <origin rpy="0 0 0" xyz="0 0 0"/>
+      <geometry>
+        <mesh filename="${mesh_prefix}assets/arms/panda/meshes/collision/link3.stl"/>
       </geometry>
     </collision>
@@ -250,14 +248,14 @@
       <origin rpy="0 0 0" xyz="0 0 0"/>
       <geometry>
-        <mesh filename="package://robot_control_assets/assets/arms/panda/meshes/visual/link4.dae"/>
-      </geometry>
-      <material name="">
-        <color rgba="1 1 1 1"/>
-      </material>
-    </visual>
-    <collision>
-      <origin rpy="0 0 0" xyz="0 0 0"/>
-      <geometry>
-        <mesh filename="package://robot_control_assets/assets/arms/panda/meshes/collision/link4.stl"/>
+        <mesh filename="${mesh_prefix}assets/arms/panda/meshes/visual/link4.dae"/>
+      </geometry>
+      <material name="">
+        <color rgba="1 1 1 1"/>
+      </material>
+    </visual>
+    <collision>
+      <origin rpy="0 0 0" xyz="0 0 0"/>
+      <geometry>
+        <mesh filename="${mesh_prefix}assets/arms/panda/meshes/collision/link4.stl"/>
       </geometry>
     </collision>
@@ -283,14 +281,14 @@
       <origin rpy="0 0 0" xyz="0 0 0"/>
       <geometry>
-        <mesh filename="package://robot_control_assets/assets/arms/panda/meshes/visual/link5.dae"/>
-      </geometry>
-      <material name="">
-        <color rgba="1 1 1 1"/>
-      </material>
-    </visual>
-    <collision>
-      <origin rpy="0 0 0" xyz="0 0 0"/>
-      <geometry>
-        <mesh filename="package://robot_control_assets/assets/arms/panda/meshes/collision/link5.stl"/>
+        <mesh filename="${mesh_prefix}assets/arms/panda/meshes/visual/link5.dae"/>
+      </geometry>
+      <material name="">
+        <color rgba="1 1 1 1"/>
+      </material>
+    </visual>
+    <collision>
+      <origin rpy="0 0 0" xyz="0 0 0"/>
+      <geometry>
+        <mesh filename="${mesh_prefix}assets/arms/panda/meshes/collision/link5.stl"/>
       </geometry>
     </collision>
@@ -314,14 +312,14 @@
       <origin rpy="0 0 0" xyz="0 0 0"/>
       <geometry>
-        <mesh filename="package://robot_control_assets/assets/arms/panda/meshes/visual/link6.dae"/>
-      </geometry>
-      <material name="">
-        <color rgba="1 1 1 1"/>
-      </material>
-    </visual>
-    <collision>
-      <origin rpy="0 0 0" xyz="0 0 0"/>
-      <geometry>
-        <mesh filename="package://robot_control_assets/assets/arms/panda/meshes/collision/link6.stl"/>
+        <mesh filename="${mesh_prefix}assets/arms/panda/meshes/visual/link6.dae"/>
+      </geometry>
+      <material name="">
+        <color rgba="1 1 1 1"/>
+      </material>
+    </visual>
+    <collision>
+      <origin rpy="0 0 0" xyz="0 0 0"/>
+      <geometry>
+        <mesh filename="${mesh_prefix}assets/arms/panda/meshes/collision/link6.stl"/>
       </geometry>
     </collision>
@@ -345,14 +343,14 @@
       <origin rpy="0 0 0" xyz="0 0 0"/>
       <geometry>
-        <mesh filename="package://robot_control_assets/assets/arms/panda/meshes/visual/link7.dae"/>
-      </geometry>
-      <material name="">
-        <color rgba="1 1 1 1"/>
-      </material>
-    </visual>
-    <collision>
-      <origin rpy="0 0 0" xyz="0 0 0"/>
-      <geometry>
-        <mesh filename="package://robot_control_assets/assets/arms/panda/meshes/collision/link7.stl"/>
+        <mesh filename="${mesh_prefix}assets/arms/panda/meshes/visual/link7.dae"/>
+      </geometry>
+      <material name="">
+        <color rgba="1 1 1 1"/>
+      </material>
+    </visual>
+    <collision>
+      <origin rpy="0 0 0" xyz="0 0 0"/>
+      <geometry>
+        <mesh filename="${mesh_prefix}assets/arms/panda/meshes/collision/link7.stl"/>
       </geometry>
     </collision>
@@ -427,14 +425,14 @@
       <origin rpy="0 0 0" xyz="0 0 0"/>
       <geometry>
-        <mesh filename="package://robot_control_assets/assets/arms/panda/meshes/visual/hand.dae"/>
-      </geometry>
-      <material name="">
-        <color rgba="1 1 1 1"/>
-      </material>
-    </visual>
-    <collision>
-      <origin rpy="0 0 0" xyz="0 0 0"/>
-      <geometry>
-        <mesh filename="package://robot_control_assets/assets/arms/panda/meshes/collision/hand.stl"/>
+        <mesh filename="${mesh_prefix}assets/arms/panda/meshes/visual/hand.dae"/>
+      </geometry>
+      <material name="">
+        <color rgba="1 1 1 1"/>
+      </material>
+    </visual>
+    <collision>
+      <origin rpy="0 0 0" xyz="0 0 0"/>
+      <geometry>
+        <mesh filename="${mesh_prefix}assets/arms/panda/meshes/collision/hand.stl"/>
       </geometry>
     </collision>
@@ -449,14 +447,14 @@
       <origin rpy="0 0 0" xyz="0 0 0"/>
       <geometry>
-        <mesh filename="package://robot_control_assets/assets/arms/panda/meshes/visual/finger.dae"/>
-      </geometry>
-      <material name="">
-        <color rgba="1 1 1 1"/>
-      </material>
-    </visual>
-    <collision>
-      <origin rpy="0 0 0" xyz="0 0 0"/>
-      <geometry>
-        <mesh filename="package://robot_control_assets/assets/arms/panda/meshes/collision/finger.stl"/>
+        <mesh filename="${mesh_prefix}assets/arms/panda/meshes/visual/finger.dae"/>
+      </geometry>
+      <material name="">
+        <color rgba="1 1 1 1"/>
+      </material>
+    </visual>
+    <collision>
+      <origin rpy="0 0 0" xyz="0 0 0"/>
+      <geometry>
+        <mesh filename="${mesh_prefix}assets/arms/panda/meshes/collision/finger.stl"/>
       </geometry>
     </collision>
@@ -471,5 +469,5 @@
       <origin rpy="0 0 3.14159265359" xyz="0 0 0"/>
       <geometry>
-        <mesh filename="package://robot_control_assets/assets/arms/panda/meshes/visual/finger.dae"/>
+        <mesh filename="${mesh_prefix}assets/arms/panda/meshes/visual/finger.dae"/>
       </geometry>
       <material name="">
@@ -480,5 +478,5 @@
       <origin rpy="0 0 3.14159265359" xyz="0 0 0"/>
       <geometry>
-        <mesh filename="package://robot_control_assets/assets/arms/panda/meshes/collision/finger.stl"/>
+        <mesh filename="${mesh_prefix}assets/arms/panda/meshes/collision/finger.stl"/>
       </geometry>
     </collision>
