Commit message: working ik controller

File: robot_control_assets/assets/arms/panda/panda.urdf.xacro (robot description, xacro)
@@ -3,9 +3,11 @@
   <xacro:property name="joint_damping" value="1.0"/>
   <xacro:arg name="mesh_prefix" default="model://" />
+  <xacro:arg name="robot_id"    default="" />
   <xacro:property name="mesh_prefix" value="$(arg mesh_prefix)" />
+  <xacro:property name="robot_id" value="$(arg robot_id)" />
   <link name="world"/>
-  <joint name="panda_joint_world" type="fixed">
+  <joint name="panda${robot_id}_joint_world" type="fixed">
     <parent link="world"/>
-    <child link="panda_link0"/>
+    <child link="panda${robot_id}_link0"/>
     <origin rpy="0 0 0" xyz="0 0 0"/>
     <dynamics damping="${joint_damping}" />
@@ -16,113 +18,113 @@
     </plugin>
   </gazebo>
-  <gazebo reference="panda_link0">
-    <material>Gazebo/White</material>
-    <mu1>0.2</mu1>
-    <mu2>0.2</mu2>
-  </gazebo>
-  <gazebo reference="panda_link1">
-    <material>Gazebo/White</material>
-    <mu1>0.2</mu1>
-    <mu2>0.2</mu2>
-  </gazebo>
-  <gazebo reference="panda_link2">
-    <material>Gazebo/White</material>
-    <mu1>0.2</mu1>
-    <mu2>0.2</mu2>
-  </gazebo>
-  <gazebo reference="panda_link3">
-    <material>Gazebo/White</material>
-    <mu1>0.2</mu1>
-    <mu2>0.2</mu2>
-  </gazebo>
-  <gazebo reference="panda_link4">
-    <material>Gazebo/White</material>
-    <mu1>0.2</mu1>
-    <mu2>0.2</mu2>
-  </gazebo>
-  <gazebo reference="panda_link5">
-    <material>Gazebo/White</material>
-    <mu1>0.2</mu1>
-    <mu2>0.2</mu2>
-  </gazebo>
-  <gazebo reference="panda_link6">
-    <material>Gazebo/White</material>
-    <mu1>0.2</mu1>
-    <mu2>0.2</mu2>
-  </gazebo>
-  <gazebo reference="panda_link7">
-    <material>Gazebo/White</material>
-    <mu1>0.2</mu1>
-    <mu2>0.2</mu2>
-  </gazebo>
-  <gazebo reference="panda_link8">
-    <material>Gazebo/White</material>
-    <mu1>0.2</mu1>
-    <mu2>0.2</mu2>
-  </gazebo>
-  <transmission name="panda_joint1_trans">
-    <type>transmission_interface/SimpleTransmission</type>
-    <joint name="panda_joint1">
-      <hardwareInterface>hardware_interface/EffortJointInterface</hardwareInterface>
-    </joint>
-    <actuator name="panda_joint1_motor">
-      <mechanicalReduction>1</mechanicalReduction>
-    </actuator>
-  </transmission>
-  <transmission name="panda_joint2_trans">
-    <type>transmission_interface/SimpleTransmission</type>
-    <joint name="panda_joint2">
-      <hardwareInterface>hardware_interface/EffortJointInterface</hardwareInterface>
-    </joint>
-    <actuator name="panda_joint2_motor">
-      <mechanicalReduction>1</mechanicalReduction>
-    </actuator>
-  </transmission>
-  <transmission name="panda_joint3_trans">
-    <type>transmission_interface/SimpleTransmission</type>
-    <joint name="panda_joint3">
-      <hardwareInterface>hardware_interface/EffortJointInterface</hardwareInterface>
-    </joint>
-    <actuator name="panda_joint3_motor">
-      <mechanicalReduction>1</mechanicalReduction>
-    </actuator>
-  </transmission>
-  <transmission name="panda_joint4_trans">
-    <type>transmission_interface/SimpleTransmission</type>
-    <joint name="panda_joint4">
-      <hardwareInterface>hardware_interface/EffortJointInterface</hardwareInterface>
-    </joint>
-    <actuator name="panda_joint4_motor">
-      <mechanicalReduction>1</mechanicalReduction>
-    </actuator>
-  </transmission>
-  <transmission name="panda_joint5_trans">
-    <type>transmission_interface/SimpleTransmission</type>
-    <joint name="panda_joint5">
-      <hardwareInterface>hardware_interface/EffortJointInterface</hardwareInterface>
-    </joint>
-    <actuator name="panda_joint5_motor">
-      <mechanicalReduction>1</mechanicalReduction>
-    </actuator>
-  </transmission>
-  <transmission name="panda_joint6_trans">
-    <type>transmission_interface/SimpleTransmission</type>
-    <joint name="panda_joint6">
-      <hardwareInterface>hardware_interface/EffortJointInterface</hardwareInterface>
-    </joint>
-    <actuator name="panda_joint6_motor">
-      <mechanicalReduction>1</mechanicalReduction>
-    </actuator>
-  </transmission>
-  <transmission name="panda_joint7_trans">
-    <type>transmission_interface/SimpleTransmission</type>
-    <joint name="panda_joint7">
-      <hardwareInterface>hardware_interface/EffortJointInterface</hardwareInterface>
-    </joint>
-    <actuator name="panda_joint7_motor">
-      <mechanicalReduction>1</mechanicalReduction>
-    </actuator>
-  </transmission>
-  <link name="panda_link0">
+  <gazebo reference="panda${robot_id}_link0">
+    <material>Gazebo/White</material>
+    <mu1>0.2</mu1>
+    <mu2>0.2</mu2>
+  </gazebo>
+  <gazebo reference="panda${robot_id}_link1">
+    <material>Gazebo/White</material>
+    <mu1>0.2</mu1>
+    <mu2>0.2</mu2>
+  </gazebo>
+  <gazebo reference="panda${robot_id}_link2">
+    <material>Gazebo/White</material>
+    <mu1>0.2</mu1>
+    <mu2>0.2</mu2>
+  </gazebo>
+  <gazebo reference="panda${robot_id}_link3">
+    <material>Gazebo/White</material>
+    <mu1>0.2</mu1>
+    <mu2>0.2</mu2>
+  </gazebo>
+  <gazebo reference="panda${robot_id}_link4">
+    <material>Gazebo/White</material>
+    <mu1>0.2</mu1>
+    <mu2>0.2</mu2>
+  </gazebo>
+  <gazebo reference="panda${robot_id}_link5">
+    <material>Gazebo/White</material>
+    <mu1>0.2</mu1>
+    <mu2>0.2</mu2>
+  </gazebo>
+  <gazebo reference="panda${robot_id}_link6">
+    <material>Gazebo/White</material>
+    <mu1>0.2</mu1>
+    <mu2>0.2</mu2>
+  </gazebo>
+  <gazebo reference="panda${robot_id}_link7">
+    <material>Gazebo/White</material>
+    <mu1>0.2</mu1>
+    <mu2>0.2</mu2>
+  </gazebo>
+  <gazebo reference="panda${robot_id}_link8">
+    <material>Gazebo/White</material>
+    <mu1>0.2</mu1>
+    <mu2>0.2</mu2>
+  </gazebo>
+  <transmission name="panda${robot_id}_joint1_trans">
+    <type>transmission_interface/SimpleTransmission</type>
+    <joint name="panda${robot_id}_joint1">
+      <hardwareInterface>hardware_interface/EffortJointInterface</hardwareInterface>
+    </joint>
+    <actuator name="panda${robot_id}_joint1_motor">
+      <mechanicalReduction>1</mechanicalReduction>
+    </actuator>
+  </transmission>
+  <transmission name="panda${robot_id}_joint2_trans">
+    <type>transmission_interface/SimpleTransmission</type>
+    <joint name="panda${robot_id}_joint2">
+      <hardwareInterface>hardware_interface/EffortJointInterface</hardwareInterface>
+    </joint>
+    <actuator name="panda${robot_id}_joint2_motor">
+      <mechanicalReduction>1</mechanicalReduction>
+    </actuator>
+  </transmission>
+  <transmission name="panda${robot_id}_joint3_trans">
+    <type>transmission_interface/SimpleTransmission</type>
+    <joint name="panda${robot_id}_joint3">
+      <hardwareInterface>hardware_interface/EffortJointInterface</hardwareInterface>
+    </joint>
+    <actuator name="panda${robot_id}_joint3_motor">
+      <mechanicalReduction>1</mechanicalReduction>
+    </actuator>
+  </transmission>
+  <transmission name="panda${robot_id}_joint4_trans">
+    <type>transmission_interface/SimpleTransmission</type>
+    <joint name="panda${robot_id}_joint4">
+      <hardwareInterface>hardware_interface/EffortJointInterface</hardwareInterface>
+    </joint>
+    <actuator name="panda${robot_id}_joint4_motor">
+      <mechanicalReduction>1</mechanicalReduction>
+    </actuator>
+  </transmission>
+  <transmission name="panda${robot_id}_joint5_trans">
+    <type>transmission_interface/SimpleTransmission</type>
+    <joint name="panda${robot_id}_joint5">
+      <hardwareInterface>hardware_interface/EffortJointInterface</hardwareInterface>
+    </joint>
+    <actuator name="panda${robot_id}_joint5_motor">
+      <mechanicalReduction>1</mechanicalReduction>
+    </actuator>
+  </transmission>
+  <transmission name="panda${robot_id}_joint6_trans">
+    <type>transmission_interface/SimpleTransmission</type>
+    <joint name="panda${robot_id}_joint6">
+      <hardwareInterface>hardware_interface/EffortJointInterface</hardwareInterface>
+    </joint>
+    <actuator name="panda${robot_id}_joint6_motor">
+      <mechanicalReduction>1</mechanicalReduction>
+    </actuator>
+  </transmission>
+  <transmission name="panda${robot_id}_joint7_trans">
+    <type>transmission_interface/SimpleTransmission</type>
+    <joint name="panda${robot_id}_joint7">
+      <hardwareInterface>hardware_interface/EffortJointInterface</hardwareInterface>
+    </joint>
+    <actuator name="panda${robot_id}_joint7_motor">
+      <mechanicalReduction>1</mechanicalReduction>
+    </actuator>
+  </transmission>
+  <link name="panda${robot_id}_link0">
     <inertial>
       <mass value="2.92"/>
@@ -146,5 +148,5 @@
     </collision>
   </link>
-  <link name="panda_link1">
+  <link name="panda${robot_id}_link1">
     <inertial>
       <mass value="2.74"/>
@@ -168,14 +170,14 @@
     </collision>
   </link>
-  <joint name="panda_joint1" type="revolute">
+  <joint name="panda${robot_id}_joint1" type="revolute">
     <safety_controller k_position="100.0" k_velocity="40.0" soft_lower_limit="-2.8973" soft_upper_limit="2.8973"/>
     <origin rpy="0 0 0" xyz="0 0 0.333"/>
-    <parent link="panda_link0"/>
-    <child link="panda_link1"/>
+    <parent link="panda${robot_id}_link0"/>
+    <child link="panda${robot_id}_link1"/>
     <axis xyz="0 0 1"/>
     <limit effort="87" lower="-2.8973" upper="2.8973" velocity="2.1750"/>
     <dynamics damping="${joint_damping}" />
   </joint>
-  <link name="panda_link2">
+  <link name="panda${robot_id}_link2">
     <inertial>
       <mass value="2.74"/>
@@ -199,14 +201,14 @@
     </collision>
   </link>
-  <joint name="panda_joint2" type="revolute">
+  <joint name="panda${robot_id}_joint2" type="revolute">
     <safety_controller k_position="100.0" k_velocity="40.0" soft_lower_limit="-1.7628" soft_upper_limit="1.7628"/>
     <origin rpy="-1.57079632679 0 0" xyz="0 0 0"/>
-    <parent link="panda_link1"/>
-    <child link="panda_link2"/>
+    <parent link="panda${robot_id}_link1"/>
+    <child link="panda${robot_id}_link2"/>
     <axis xyz="0 0 1"/>
     <limit effort="87" lower="-1.7628" upper="1.7628" velocity="2.1750"/>
     <dynamics damping="${joint_damping}" />
   </joint>
-  <link name="panda_link3">
+  <link name="panda${robot_id}_link3">
     <inertial>
       <mass value="2.38"/>
@@ -230,14 +232,14 @@
     </collision>
   </link>
-  <joint name="panda_joint3" type="revolute">
+  <joint name="panda${robot_id}_joint3" type="revolute">
     <safety_controller k_position="100.0" k_velocity="40.0" soft_lower_limit="-2.8973" soft_upper_limit="2.8973"/>
     <origin rpy="1.57079632679 0 0" xyz="0 -0.316 0"/>
-    <parent link="panda_link2"/>
-    <child link="panda_link3"/>
+    <parent link="panda${robot_id}_link2"/>
+    <child link="panda${robot_id}_link3"/>
     <axis xyz="0 0 1"/>
     <limit effort="87" lower="-2.8973" upper="2.8973" velocity="2.1750"/>
     <dynamics damping="${joint_damping}" />
   </joint>
-  <link name="panda_link4">
+  <link name="panda${robot_id}_link4">
     <inertial>
       <mass value="2.38"/>
@@ -261,10 +263,10 @@
     </collision>
   </link>
-  <joint name="panda_joint4" type="revolute">
+  <joint name="panda${robot_id}_joint4" type="revolute">
     <safety_controller k_position="100.0" k_velocity="40.0" soft_lower_limit="-3.0718" soft_upper_limit="0.0698"/>
     <!-- soft_upper_limitr should be -0.0698, but that brakes simulation when initial position for this joint is 0.0 -->
     <origin rpy="1.57079632679 0 0" xyz="0.0825 0 0"/>
-    <parent link="panda_link3"/>
-    <child link="panda_link4"/>
+    <parent link="panda${robot_id}_link3"/>
+    <child link="panda${robot_id}_link4"/>
     <axis xyz="0 0 1"/>
     <limit effort="87" lower="-3.0718" upper="0.0698" velocity="2.1750"/>
@@ -272,5 +274,5 @@
     <dynamics damping="${joint_damping}" />
   </joint>
-  <link name="panda_link5">
+  <link name="panda${robot_id}_link5">
     <inertial>
       <mass value="2.74"/>
@@ -294,14 +296,14 @@
     </collision>
   </link>
-  <joint name="panda_joint5" type="revolute">
+  <joint name="panda${robot_id}_joint5" type="revolute">
     <safety_controller k_position="100.0" k_velocity="40.0" soft_lower_limit="-2.8973" soft_upper_limit="2.8973"/>
     <origin rpy="-1.57079632679 0 0" xyz="-0.0825 0.384 0"/>
-    <parent link="panda_link4"/>
-    <child link="panda_link5"/>
+    <parent link="panda${robot_id}_link4"/>
+    <child link="panda${robot_id}_link5"/>
     <axis xyz="0 0 1"/>
     <limit effort="12" lower="-2.8973" upper="2.8973" velocity="2.6100"/>
     <dynamics damping="${joint_damping}" />
   </joint>
-  <link name="panda_link6">
+  <link name="panda${robot_id}_link6">
     <inertial>
       <mass value="1.55"/>
@@ -325,14 +327,14 @@
     </collision>
   </link>
-  <joint name="panda_joint6" type="revolute">
+  <joint name="panda${robot_id}_joint6" type="revolute">
     <safety_controller k_position="100.0" k_velocity="40.0" soft_lower_limit="-0.0175" soft_upper_limit="3.7525"/>
     <origin rpy="1.57079632679 0 0" xyz="0 0 0"/>
-    <parent link="panda_link5"/>
-    <child link="panda_link6"/>
+    <parent link="panda${robot_id}_link5"/>
+    <child link="panda${robot_id}_link6"/>
     <axis xyz="0 0 1"/>
     <limit effort="12" lower="-0.0175" upper="3.7525" velocity="2.6100"/>
     <dynamics damping="${joint_damping}" />
   </joint>
-  <link name="panda_link7">
+  <link name="panda${robot_id}_link7">
     <inertial>
       <mass value="0.54"/>
@@ -356,14 +358,14 @@
     </collision>
   </link>
-  <joint name="panda_joint7" type="revolute">
+  <joint name="panda${robot_id}_joint7" type="revolute">
     <safety_controller k_position="100.0" k_velocity="40.0" soft_lower_limit="-2.8973" soft_upper_limit="2.8973"/>
     <origin rpy="1.57079632679 0 0" xyz="0.088 0 0"/>
-    <parent link="panda_link6"/>
-    <child link="panda_link7"/>
+    <parent link="panda${robot_id}_link6"/>
+    <child link="panda${robot_id}_link7"/>
     <axis xyz="0 0 1"/>
     <limit effort="12" lower="-2.8973" upper="2.8973" velocity="2.6100"/>
     <dynamics damping="${joint_damping}" />
   </joint>
-  <link name="panda_link8">
+  <link name="panda${robot_id}_link8">
     <inertial>
       <mass value="0.0"/>
@@ -372,49 +374,49 @@
     </inertial>
   </link>
-  <joint name="panda_joint8" type="fixed">
+  <joint name="panda${robot_id}_joint8" type="fixed">
     <origin rpy="0 0 0" xyz="0 0 0.107"/>
-    <parent link="panda_link7"/>
-    <child link="panda_link8"/>
+    <parent link="panda${robot_id}_link7"/>
+    <child link="panda${robot_id}_link8"/>
     <axis xyz="0 0 0"/>
   </joint>
-  <joint name="panda_hand_joint" type="fixed">
-    <parent link="panda_link8"/>
-    <child link="panda_hand"/>
+  <joint name="panda${robot_id}_hand_joint" type="fixed">
+    <parent link="panda${robot_id}_link8"/>
+    <child link="panda${robot_id}_hand"/>
     <origin rpy="0 0 -0.785398163397" xyz="0 0 0"/>
   </joint>
-  <gazebo reference="panda_hand">
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