Commit message: working controller on both kinova and panda

File: robot_control_assets/assets/arms/kinova3/kinova3.urdf.xacro (robot description, xacro)
@@ -1,4 +1,12 @@
 <?xml version="1.0" encoding="utf-8"?>
-<robot name="kinova3">
+<robot name="kinova3" xmlns:xacro="http://www.ros.org/wiki/xacro">
+  <xacro:arg name="mesh_prefix" default="model://" />
+  <xacro:property name="mesh_prefix" value="$(arg mesh_prefix)" />
+  <link name="world"/>
+  <joint name="world_base_joint" type="fixed">
+    <origin rpy="0 0 0" xyz="0 0 0"/>
+    <parent link="world"/>
+    <child link="base_link"/>
+  </joint>
   <link name="base_link">
     <!-- <inertial>
@@ -10,14 +18,14 @@
       <origin rpy="0 0 0" xyz="0 0 0"/>
       <geometry>
-        <mesh filename="package://robot_control/assets/arms/kinova3/meshes/base_link.STL"/>
-      </geometry>
-      <material name="">
-        <color rgba="0.75294 0.75294 0.75294 1"/>
-      </material>
-    </visual>
-    <collision>
-      <origin rpy="0 0 0" xyz="0 0 0"/>
-      <geometry>
-        <mesh filename="package://robot_control/assets/arms/kinova3/meshes/base_link.STL"/>
+        <mesh filename="${mesh_prefix}assets/arms/kinova3/meshes/base_link.STL"/>
+      </geometry>
+      <material name="">
+        <color rgba="0.75294 0.75294 0.75294 1"/>
+      </material>
+    </visual>
+    <collision>
+      <origin rpy="0 0 0" xyz="0 0 0"/>
+      <geometry>
+        <mesh filename="${mesh_prefix}assets/arms/kinova3/meshes/base_link.STL"/>
       </geometry>
     </collision>`
@@ -44,14 +52,14 @@
       <origin rpy="0 0 0" xyz="0 0 0"/>
       <geometry>
-        <mesh filename="package://robot_control/assets/arms/kinova3/meshes/shoulder_link.STL"/>
-      </geometry>
-      <material name="">
-        <color rgba="0.75294 0.75294 0.75294 1"/>
-      </material>
-    </visual>
-    <collision>
-      <origin rpy="0 0 0" xyz="0 0 0"/>
-      <geometry>
-        <mesh filename="package://robot_control/assets/arms/kinova3/meshes/shoulder_link.STL"/>
+        <mesh filename="${mesh_prefix}assets/arms/kinova3/meshes/shoulder_link.STL"/>
+      </geometry>
+      <material name="">
+        <color rgba="0.75294 0.75294 0.75294 1"/>
+      </material>
+    </visual>
+    <collision>
+      <origin rpy="0 0 0" xyz="0 0 0"/>
+      <geometry>
+        <mesh filename="${mesh_prefix}assets/arms/kinova3/meshes/shoulder_link.STL"/>
       </geometry>
     </collision>
@@ -62,5 +70,5 @@
     <child link="shoulder_link"/>
     <axis xyz="0 0 1"/>
-    <limit effort="39" velocity="1.3963"  upper="3.14" lower="-3.14"/>
+    <limit effort="39" velocity="1.3963"  upper="3.17" lower="-3.17"/>
   </joint>
   <link name="half_arm_1_link">
@@ -73,14 +81,14 @@
       <origin rpy="0 0 0" xyz="0 0 0"/>
       <geometry>
-        <mesh filename="package://robot_control/assets/arms/kinova3/meshes/half_arm_1_link.STL"/>
-      </geometry>
-      <material name="">
-        <color rgba="0.75294 0.75294 0.75294 1"/>
-      </material>
-    </visual>
-    <collision>
-      <origin rpy="0 0 0" xyz="0 0 0"/>
-      <geometry>
-        <mesh filename="package://robot_control/assets/arms/kinova3/meshes/half_arm_1_link.STL"/>
+        <mesh filename="${mesh_prefix}assets/arms/kinova3/meshes/half_arm_1_link.STL"/>
+      </geometry>
+      <material name="">
+        <color rgba="0.75294 0.75294 0.75294 1"/>
+      </material>
+    </visual>
+    <collision>
+      <origin rpy="0 0 0" xyz="0 0 0"/>
+      <geometry>
+        <mesh filename="${mesh_prefix}assets/arms/kinova3/meshes/half_arm_1_link.STL"/>
       </geometry>
     </collision>
@@ -102,14 +110,14 @@
       <origin rpy="0 0 0" xyz="0 0 0"/>
       <geometry>
-        <mesh filename="package://robot_control/assets/arms/kinova3/meshes/half_arm_2_link.STL"/>
-      </geometry>
-      <material name="">
-        <color rgba="0.75294 0.75294 0.75294 1"/>
-      </material>
-    </visual>
-    <collision>
-      <origin rpy="0 0 0" xyz="0 0 0"/>
-      <geometry>
-        <mesh filename="package://robot_control/assets/arms/kinova3/meshes/half_arm_2_link.STL"/>
+        <mesh filename="${mesh_prefix}assets/arms/kinova3/meshes/half_arm_2_link.STL"/>
+      </geometry>
+      <material name="">
+        <color rgba="0.75294 0.75294 0.75294 1"/>
+      </material>
+    </visual>
+    <collision>
+      <origin rpy="0 0 0" xyz="0 0 0"/>
+      <geometry>
+        <mesh filename="${mesh_prefix}assets/arms/kinova3/meshes/half_arm_2_link.STL"/>
       </geometry>
     </collision>
@@ -120,5 +128,5 @@
     <child link="half_arm_2_link"/>
     <axis xyz="0 0 1"/>
-    <limit effort="39" velocity="1.3963"    upper="3.14" lower="-3.14"/>
+    <limit effort="39" velocity="1.3963"    upper="3.17" lower="-3.17"/>
   </joint>
   <link name="forearm_link">
@@ -131,14 +139,14 @@
       <origin rpy="0 0 0" xyz="0 0 0"/>
       <geometry>
-        <mesh filename="package://robot_control/assets/arms/kinova3/meshes/forearm_link.STL"/>
-      </geometry>
-      <material name="">
-        <color rgba="0.75294 0.75294 0.75294 1"/>
-      </material>
-    </visual>
-    <collision>
-      <origin rpy="0 0 0" xyz="0 0 0"/>
-      <geometry>
-        <mesh filename="package://robot_control/assets/arms/kinova3/meshes/forearm_link.STL"/>
+        <mesh filename="${mesh_prefix}assets/arms/kinova3/meshes/forearm_link.STL"/>
+      </geometry>
+      <material name="">
+        <color rgba="0.75294 0.75294 0.75294 1"/>
+      </material>
+    </visual>
+    <collision>
+      <origin rpy="0 0 0" xyz="0 0 0"/>
+      <geometry>
+        <mesh filename="${mesh_prefix}assets/arms/kinova3/meshes/forearm_link.STL"/>
       </geometry>
     </collision>
@@ -160,14 +168,14 @@
       <origin rpy="0 0 0" xyz="0 0 0"/>
       <geometry>
-        <mesh filename="package://robot_control/assets/arms/kinova3/meshes/spherical_wrist_1_link.STL"/>
-      </geometry>
-      <material name="">
-        <color rgba="0.75294 0.75294 0.75294 1"/>
-      </material>
-    </visual>
-    <collision>
-      <origin rpy="0 0 0" xyz="0 0 0"/>
-      <geometry>
-        <mesh filename="package://robot_control/assets/arms/kinova3/meshes/spherical_wrist_1_link.STL"/>
+        <mesh filename="${mesh_prefix}assets/arms/kinova3/meshes/spherical_wrist_1_link.STL"/>
+      </geometry>
+      <material name="">
+        <color rgba="0.75294 0.75294 0.75294 1"/>
+      </material>
+    </visual>
+    <collision>
+      <origin rpy="0 0 0" xyz="0 0 0"/>
+      <geometry>
+        <mesh filename="${mesh_prefix}assets/arms/kinova3/meshes/spherical_wrist_1_link.STL"/>
       </geometry>
     </collision>
@@ -178,5 +186,5 @@
     <child link="spherical_wrist_1_link"/>
     <axis xyz="0 0 1"/>
-    <limit effort="9" velocity="1.2218"    upper="3.14" lower="-3.14"/>
+    <limit effort="9" velocity="1.2218"    upper="3.17" lower="-3.17"/>
   </joint>
   <link name="spherical_wrist_2_link">
@@ -189,14 +197,14 @@
       <origin rpy="0 0 0" xyz="0 0 0"/>
       <geometry>
-        <mesh filename="package://robot_control/assets/arms/kinova3/meshes/spherical_wrist_2_link.STL"/>
-      </geometry>
-      <material name="">
-        <color rgba="0.75294 0.75294 0.75294 1"/>
-      </material>
-    </visual>
-    <collision>
-      <origin rpy="0 0 0" xyz="0 0 0"/>
-      <geometry>
-        <mesh filename="package://robot_control/assets/arms/kinova3/meshes/spherical_wrist_2_link.STL"/>
+        <mesh filename="${mesh_prefix}assets/arms/kinova3/meshes/spherical_wrist_2_link.STL"/>
+      </geometry>
+      <material name="">
+        <color rgba="0.75294 0.75294 0.75294 1"/>
+      </material>
+    </visual>
+    <collision>
+      <origin rpy="0 0 0" xyz="0 0 0"/>
+      <geometry>
+        <mesh filename="${mesh_prefix}assets/arms/kinova3/meshes/spherical_wrist_2_link.STL"/>
       </geometry>
     </collision>
@@ -218,14 +226,14 @@
       <origin rpy="0 0 0" xyz="0 0 0"/>
       <geometry>
-        <mesh filename="package://robot_control/assets/arms/kinova3/meshes/bracelet_with_vision_link.STL"/>
-      </geometry>
-      <material name="">
-        <color rgba="0.75294 0.75294 0.75294 1"/>
-      </material>
-    </visual>
-    <collision>
-      <origin rpy="0 0 0" xyz="0 0 0"/>
-      <geometry>
-        <mesh filename="package://robot_control/assets/arms/kinova3/meshes/bracelet_with_vision_link.STL"/>
+        <mesh filename="${mesh_prefix}assets/arms/kinova3/meshes/bracelet_with_vision_link.STL"/>
+      </geometry>
+      <material name="">
+        <color rgba="0.75294 0.75294 0.75294 1"/>
+      </material>
+    </visual>
+    <collision>
+      <origin rpy="0 0 0" xyz="0 0 0"/>
+      <geometry>
+        <mesh filename="${mesh_prefix}assets/arms/kinova3/meshes/bracelet_with_vision_link.STL"/>
       </geometry>
     </collision>
@@ -236,5 +244,5 @@
     <child link="bracelet_link"/>
     <axis xyz="0 0 1"/>
-    <limit effort="9" velocity="1.2218"   upper="3.14" lower="-3.14"/>
+    <limit effort="9" velocity="1.2218"   upper="3.17" lower="-3.17"/>
   </joint>
   <link name="end_effector_link">
@@ -251,3 +259,72 @@
     <axis xyz="0 0 0"/>
   </joint>
+  <transmission name="joint_1_transmission">
+    <type>transmission_interface/SimpleTransmission</type>
+    <joint name="joint_1">
+      <hardwareInterface>hardware_interface/EffortJointInterface</hardwareInterface>
+    </joint>
+    <actuator name="joint_1_motor">
+      <mechanicalReduction>1</mechanicalReduction>
+    </actuator>
+  </transmission>
+  <transmission name="joint_2_transmission">
+    <type>transmission_interface/SimpleTransmission</type>
+    <joint name="joint_2">
+      <hardwareInterface>hardware_interface/EffortJointInterface</hardwareInterface>
+    </joint>
+    <actuator name="joint_2_motor">
+      <mechanicalReduction>1</mechanicalReduction>
+    </actuator>
+  </transmission>
+  <transmission name="joint_3_transmission">
+    <type>transmission_interface/SimpleTransmission</type>
+    <joint name="joint_3">
+      <hardwareInterface>hardware_interface/EffortJointInterface</hardwareInterface>
+    </joint>
+    <actuator name="joint_3_motor">
+      <mechanicalReduction>1</mechanicalReduction>
+    </actuator>
+  </transmission>
+  <transmission name="joint_4_transmission">
+    <type>transmission_interface/SimpleTransmission</type>
+    <joint name="joint_4">
+      <hardwareInterface>hardware_interface/EffortJointInterface</hardwareInterface>
+    </joint>
+    <actuator name="joint_4_motor">
+      <mechanicalReduction>1</mechanicalReduction>
+    </actuator>
+  </transmission>
+  <transmission name="joint_5_transmission">
+    <type>transmission_interface/SimpleTransmission</type>
+    <joint name="joint_5">
+      <hardwareInterface>hardware_interface/EffortJointInterface</hardwareInterface>
+    </joint>
+    <actuator name="joint_5_motor">
+      <mechanicalReduction>1</mechanicalReduction>
+    </actuator>
+  </transmission>
+  <transmission name="joint_6_transmission">
+    <type>transmission_interface/SimpleTransmission</type>
+    <joint name="joint_6">
+      <hardwareInterface>hardware_interface/EffortJointInterface</hardwareInterface>
+    </joint>
+    <actuator name="joint_6_motor">
+      <mechanicalReduction>1</mechanicalReduction>
+    </actuator>
+  </transmission>
+  <transmission name="joint_7_transmission">
+    <type>transmission_interface/SimpleTransmission</type>
+    <joint name="joint_7">
+      <hardwareInterface>hardware_interface/EffortJointInterface</hardwareInterface>
+    </joint>
+    <actuator name="joint_7_motor">
+      <mechanicalReduction>1</mechanicalReduction>
+    </actuator>
+  </transmission>
+  <gazebo>
+    <plugin name="gazebo_ros_control" filename="libgazebo_ros_control.so">
+      <legacyModeNS>true</legacyModeNS>
+      <!--robotParam>kinova_no_finger</robotParam-->
+    </plugin>
+  </gazebo>
 </robot>

Commit message: more changes

File: robot_control_assets/assets/arms/kinova3/kinova3.urdf.xacro (robot description, xacro)
@@ -70,5 +70,5 @@
     <child link="shoulder_link"/>
     <axis xyz="0 0 1"/>
-    <limit effort="39" velocity="1.3963"  upper="3.17" lower="-3.17"/>
+    <limit effort="39" velocity="1.3963"  upper="6.28" lower="-6.28"/>
   </joint>
   <link name="half_arm_1_link">
@@ -128,5 +128,5 @@
     <child link="half_arm_2_link"/>
     <axis xyz="0 0 1"/>
-    <limit effort="39" velocity="1.3963"    upper="3.17" lower="-3.17"/>
+    <limit effort="39" velocity="1.3963"    upper="6.28" lower="-6.28"/>
   </joint>
   <link name="forearm_link">
@@ -186,5 +186,5 @@
     <child link="spherical_wrist_1_link"/>
     <axis xyz="0 0 1"/>
-    <limit effort="9" velocity="1.2218"    upper="3.17" lower="-3.17"/>
+    <limit effort="9" velocity="1.2218"    upper="6.28" lower="-6.28"/>
   </joint>
   <link name="spherical_wrist_2_link">
@@ -244,5 +244,5 @@
     <child link="bracelet_link"/>
     <axis xyz="0 0 1"/>
-    <limit effort="9" velocity="1.2218"   upper="3.17" lower="-3.17"/>
+    <limit effort="9" velocity="1.2218"   upper="6.28" lower="-6.28"/>
   </joint>
   <link name="end_effector_link">
