Commit message: loading the object and valve fix

File: robot_control_assets/assets/objects/valve/valve.urdf.xacro (robot description, xacro)
@@ -62,3 +62,20 @@
     <limit effort="30" velocity="1.0" lower="-3.14" upper="3.14"/>
   </joint>
+  <!-- Gazebo simulation -->
+  <transmission name="wheel_joint_transmission">
+    <type>transmission_interface/SimpleTransmission</type>
+    <joint name="wheel_joint">
+      <hardwareInterface>hardware_interface/EffortJointInterface</hardwareInterface>
+    </joint>
+    <actuator name="wheel_joint_motor">
+      <mechanicalReduction>1</mechanicalReduction>
+    </actuator>
+  </transmission>
+  <gazebo>
+    <plugin name="gazebo_ros_control" filename="libgazebo_ros_control.so">
+      <legacyModeNS>true</legacyModeNS>
+      <robotParam>valve_description</robotParam>
+      <robotNamespace>valve</robotNamespace>
+    </plugin>
+  </gazebo>
 </robot>

Commit message: flag set at start and current joint target publisher

File: robot_control_assets/assets/objects/valve/valve.urdf.xacro (robot description, xacro)
@@ -59,5 +59,5 @@
     <parent link="valve_base"/>
     <child link="wheel"/>
-    <dynamics damping="1.0" friction="10.0"/>
+    <dynamics damping="10.0" friction="10.0"/>
     <limit effort="30" velocity="1.0" lower="-3.14" upper="3.14"/>
   </joint>
